Commit message: Contact sensor working partially

File: urdf/plugin.gazebo.xacro (robot description, xacro)
@@ -6,4 +6,38 @@
       <robotSimType>cob_gazebo_ros_control/HWISwitchRobotHWSim</robotSimType>
     </plugin>
+  </gazebo>
+  <gazebo reference="robotiq_85_right_finger_tip_link">
+      <sensor name="main_bumper" type="contact">
+          <geom>robotiq_85_right_finger_tip_link_geom</geom>
+          <selfCollide>true</selfCollide>
+          <alwaysOn>true</alwaysOn>
+          <updateRate>15.0</updateRate>
+          <material>Gazebo/Red</material>
+          <contact>
+            <!-- The name within the <collision> element must be of the form <link name>_collision -->
+             <collision>robotiq_85_right_finger_tip_link_collision</collision>
+          </contact>
+          <plugin name="gazebo_ros_bumper_controller" filename="libgazebo_ros_bumper.so">
+              <bumperTopicName>right_finger_bumper_vals</bumperTopicName>
+              <frameName>robotiq_85_right_finger_tip_link</frameName>
+          </plugin>
+      </sensor>
+  </gazebo>
+  <gazebo reference="robotiq_85_left_finger_tip_link">
+      <sensor name="main_bumper" type="contact">
+          <geom>robotiq_85_left_finger_tip_link_geom</geom>
+          <selfCollide>true</selfCollide>
+          <alwaysOn>true</alwaysOn>
+          <updateRate>15.0</updateRate>
+          <material>Gazebo/Red</material>
+          <contact>
+            <!-- The name within the <collision> element must be of the form <link name>_collision -->
+             <collision>robotiq_85_left_finger_tip_link_collision</collision>
+          </contact>
+          <plugin name="gazebo_ros_bumper_controller" filename="libgazebo_ros_bumper.so">
+              <bumperTopicName>left_finger_bumper_vals</bumperTopicName>
+              <frameName>robotiq_85_left_finger_tip_link</frameName>
+          </plugin>
+      </sensor>
   </gazebo>
   <!-- <gazebo reference="robotiq_85_left_inner_knuckle_link">
@@ -73,5 +107,5 @@
     <minDepth>0.01</minDepth>
   </gazebo> -->
-  <gazebo reference="box_link">
+  <!-- <gazebo reference="box_link">
     <implicitSpringDamper>1</implicitSpringDamper>
     <kp>100000.0</kp>
@@ -81,5 +115,5 @@
     <fdir1>1 0 0</fdir1>
     <minDepth>0.01</minDepth>
-  </gazebo>
+  </gazebo> -->
   <!-- camera -->
   <!-- <gazebo reference="CAM_support_link">

File: urdf/ur5_with_cam.urdf.xacro (robot description, xacro)
@@ -104,5 +104,5 @@
     <provideFeedback>true</provideFeedback>
   </gazebo>
-  <gazebo>
+  <!-- <gazebo>
     <plugin name="ft_sensor_plugin" filename="libgazebo_ros_ft_sensor.so">
       <updateRate>250.0</updateRate>
@@ -111,5 +111,5 @@
       <jointName>wrist_3_joint</jointName>
     </plugin>
-  </gazebo>
+   </gazebo>-->
   <!-- <gazebo>
     <gripper name="gazebo_gripper">
