Commit message: pkg name update

File: urdf/_d435.urdf.xacro (robot description, xacro)
@@ -8,5 +8,5 @@
 <robot name="sensor_d435" xmlns:xacro="http://ros.org/wiki/xacro">
   <!--File includes-->
-  <xacro:include filename="$(find real-time-grasp)/urdf/_d435.gazebo.xacro"/>
+  <xacro:include filename="$(find real_time_grasp)/urdf/_d435.gazebo.xacro"/>
   <xacro:macro name="sensor_d435" params="name:=camera topics_ns:=camera parent *origin">
     <xacro:property name="M_PI" value="3.1415926535897931" />

File: urdf/ur5_with_cam.urdf.xacro (robot description, xacro)
@@ -5,12 +5,12 @@
   <xacro:arg name="load_table" default="false"/>
   <!-- Gazebo plugin -->
-  <xacro:include filename="$(find real-time-grasp)/urdf/plugin.gazebo.xacro"/>
+  <xacro:include filename="$(find real_time_grasp)/urdf/plugin.gazebo.xacro"/>
   <!-- Robotiq gripper -->
   <xacro:include filename="$(find robotiq_description)/urdf/robotiq_85_gripper.urdf.xacro"/>
   <!-- ur5 -->
-  <xacro:include filename="$(find real-time-grasp)/urdf/ur5.urdf.xacro"/>
+  <xacro:include filename="$(find real_time_grasp)/urdf/ur5.urdf.xacro"/>
   <!-- It is necessary to change the hardware interface on the fly -->
-  <xacro:include filename="$(find real-time-grasp)/urdf/ur5.transmission.xacro"/>
-  <xacro:include filename="$(find real-time-grasp)/urdf/_d435.urdf.xacro" />
+  <xacro:include filename="$(find real_time_grasp)/urdf/ur5.transmission.xacro"/>
+  <xacro:include filename="$(find real_time_grasp)/urdf/_d435.urdf.xacro" />
   <!-- arm -->
   <xacro:ur5_robot prefix="" joint_limited="false" transmission_hw_interface="$(arg transmission_hw_interface)"/>
@@ -48,5 +48,5 @@
       <origin rpy="${1.57 - 0.244} ${3.14} -1.57" xyz="${0.002 - 0.03} ${-0.023 + 0.03 - 0.01} ${0.13915-0.205}"/>
       <geometry>
-        <mesh filename="package://real-time-grasp/models/cam_support/CAM_support.STL" scale="0.001 0.001 0.001"/>
+        <mesh filename="package://real_time_grasp/models/cam_support/CAM_support.STL" scale="0.001 0.001 0.001"/>
       </geometry>
       <material name="Cyan">

Commit message: Organizing repo

File: urdf/_d435.urdf.xacro (robot description, xacro)
@@ -8,5 +8,5 @@
 <robot name="sensor_d435" xmlns:xacro="http://ros.org/wiki/xacro">
   <!--File includes-->
-  <xacro:include filename="$(find real_time_grasp)/urdf/_d435.gazebo.xacro"/>
+  <xacro:include filename="$(find ssggcnn_ur5_grasping)/urdf/_d435.gazebo.xacro"/>
   <xacro:macro name="sensor_d435" params="name:=camera topics_ns:=camera parent *origin">
     <xacro:property name="M_PI" value="3.1415926535897931" />

File: urdf/ur5_with_cam.urdf.xacro (robot description, xacro)
@@ -5,12 +5,12 @@
   <xacro:arg name="load_table" default="false"/>
   <!-- Gazebo plugin -->
-  <xacro:include filename="$(find real_time_grasp)/urdf/plugin.gazebo.xacro"/>
+  <xacro:include filename="$(find ssggcnn_ur5_grasping)/urdf/plugin.gazebo.xacro"/>
   <!-- Robotiq gripper -->
   <xacro:include filename="$(find robotiq_description)/urdf/robotiq_85_gripper.urdf.xacro"/>
   <!-- ur5 -->
-  <xacro:include filename="$(find real_time_grasp)/urdf/ur5.urdf.xacro"/>
+  <xacro:include filename="$(find ssggcnn_ur5_grasping)/urdf/ur5.urdf.xacro"/>
   <!-- It is necessary to change the hardware interface on the fly -->
-  <xacro:include filename="$(find real_time_grasp)/urdf/ur5.transmission.xacro"/>
-  <xacro:include filename="$(find real_time_grasp)/urdf/_d435.urdf.xacro" />
+  <xacro:include filename="$(find ssggcnn_ur5_grasping)/urdf/ur5.transmission.xacro"/>
+  <xacro:include filename="$(find ssggcnn_ur5_grasping)/urdf/_d435.urdf.xacro" />
   <!-- arm -->
   <xacro:ur5_robot prefix="" joint_limited="false" transmission_hw_interface="$(arg transmission_hw_interface)"/>
@@ -47,5 +47,5 @@
       <origin rpy="${1.57 - 0.244} ${3.14} -1.57" xyz="${0.002 - 0.03} ${-0.023 + 0.03 - 0.01} ${0.13915-0.205}"/>
       <geometry>
-        <mesh filename="package://real_time_grasp/models/cam_support/CAM_support.STL" scale="0.001 0.001 0.001"/>
+        <mesh filename="package://ssggcnn_ur5_grasping/models/cam_support/CAM_support.STL" scale="0.001 0.001 0.001"/>
       </geometry>
       <material name="Cyan">
